Commit message: update ridgeback meshes

File: ridgeback_manipulation_description/urdf/hams.urdf.xacro (robot description, xacro)
@@ -1,5 +1,5 @@
 <?xml version="1.0"?>
 <robot xmlns:xacro="http://ros.org/wiki/xacro">
-<xacro:property name="pi" value="3.1415926535897931" />
+  <xacro:property name="pi" value="3.1415926535897931" />
   <!--link name="table_top_link">
     <visual>
