Commit message: Update iiwa description

File: ridgeback_iiwa_description/urdf/iiwa7.xacro (robot description, xacro)
@@ -2,9 +2,9 @@
 <robot xmlns:xacro="http://www.ros.org/wiki/xacro">
   <!-- Import all Gazebo-customization elements, including Gazebo colors -->
-  <xacro:include filename="$(find ridgeback_iiwa_description)/urdf/iiwa.gazebo.xacro" />
+  <xacro:include filename="$(find iiwa_description)/urdf/iiwa.gazebo.xacro" />
   <!-- Import Transmissions -->
-  <xacro:include filename="$(find ridgeback_iiwa_description)/urdf/iiwa.transmission.xacro" />
+  <xacro:include filename="$(find iiwa_description)/urdf/iiwa.transmission.xacro" />
   <!-- Include Utilities -->
-  <xacro:include filename="$(find ridgeback_iiwa_description)/urdf/utilities.xacro" />
+  <xacro:include filename="$(find iiwa_description)/urdf/utilities.xacro" />
   <!-- some constants -->
   <xacro:property name="safety_controller_k_pos" value="100" />
@@ -29,7 +29,6 @@
         <origin xyz="0 0 0" rpy="0 0 0"/>
         <geometry>
-          <mesh filename="package://iiwa_description/meshes/iiwa7/visual/link_0.stl"/>
-        </geometry>
-        <material name="Grey"/>
+          <mesh filename="package://iiwa_description/meshes/iiwa7/visual/link_0.dae"/>
+        </geometry>
       </visual>
       <collision>
@@ -38,5 +37,4 @@
           <mesh filename="package://iiwa_description/meshes/iiwa7/collision/link_0.stl"/>
         </geometry>
-        <material name="Grey"/>
       </collision>
       <self_collision_checking>
@@ -70,7 +68,6 @@
         <origin xyz="0 0 0.0075" rpy="0 0 0"/>
         <geometry>
-          <mesh filename="package://iiwa_description/meshes/iiwa7/visual/link_1.stl"/>
-        </geometry>
-        <material name="Orange"/>
+          <mesh filename="package://iiwa_description/meshes/iiwa7/visual/link_1.dae"/>
+        </geometry>
       </visual>
       <collision>
@@ -79,5 +76,4 @@
           <mesh filename="package://iiwa_description/meshes/iiwa7/collision/link_1.stl"/>
         </geometry>
-        <material name="Orange"/>
       </collision>
     </link>
@@ -104,7 +100,6 @@
         <origin xyz="0 0 0" rpy="0 0 0"/>
         <geometry>
-          <mesh filename="package://iiwa_description/meshes/iiwa7/visual/link_2.stl"/>
-        </geometry>
-        <material name="Orange"/>
+          <mesh filename="package://iiwa_description/meshes/iiwa7/visual/link_2.dae"/>
+        </geometry>
       </visual>
       <collision>
@@ -113,5 +108,4 @@
           <mesh filename="package://iiwa_description/meshes/iiwa7/collision/link_2.stl"/>
         </geometry>
-        <material name="Orange"/>
       </collision>
     </link>
@@ -138,7 +132,6 @@
         <origin xyz="0 0 -0.026" rpy="0 0 0"/>
         <geometry>
-          <mesh filename="package://iiwa_description/meshes/iiwa7/visual/link_3.stl"/>
-        </geometry>
-        <material name="Orange"/>
+          <mesh filename="package://iiwa_description/meshes/iiwa7/visual/link_3.dae"/>
+        </geometry>
       </visual>
       <collision>
@@ -147,5 +140,4 @@
           <mesh filename="package://iiwa_description/meshes/iiwa7/collision/link_3.stl"/>
         </geometry>
-        <material name="Orange"/>
       </collision>
     </link>
@@ -172,7 +164,6 @@
         <origin xyz="0 0 0" rpy="0 0 0"/>
         <geometry>
-          <mesh filename="package://iiwa_description/meshes/iiwa7/visual/link_4.stl"/>
-        </geometry>
-        <material name="Orange"/>
+          <mesh filename="package://iiwa_description/meshes/iiwa7/visual/link_4.dae"/>
+        </geometry>
       </visual>
       <collision>
@@ -181,5 +172,4 @@
           <mesh filename="package://iiwa_description/meshes/iiwa7/collision/link_4.stl"/>
         </geometry>
-        <material name="Orange"/>
       </collision>
     </link>
@@ -206,7 +196,6 @@
         <origin xyz="0 0 -0.026" rpy="0 0 0"/>
         <geometry>
-          <mesh filename="package://iiwa_description/meshes/iiwa7/visual/link_5.stl"/>
-        </geometry>
-        <material name="Orange"/>
+          <mesh filename="package://iiwa_description/meshes/iiwa7/visual/link_5.dae"/>
+        </geometry>
       </visual>
       <collision>
@@ -215,5 +204,4 @@
           <mesh filename="package://iiwa_description/meshes/iiwa7/collision/link_5.stl"/>
         </geometry>
-        <material name="Orange"/>
       </collision>
     </link>
@@ -240,7 +228,6 @@
         <origin xyz="0 0 0" rpy="0 0 0"/>
         <geometry>
-          <mesh filename="package://iiwa_description/meshes/iiwa7/visual/link_6.stl"/>
-        </geometry>
-        <material name="Orange"/>
+          <mesh filename="package://iiwa_description/meshes/iiwa7/visual/link_6.dae"/>
+        </geometry>
       </visual>
       <collision>
@@ -249,5 +236,4 @@
           <mesh filename="package://iiwa_description/meshes/iiwa7/collision/link_6.stl"/>
         </geometry>
-        <material name="Orange"/>
       </collision>
     </link>
