Commit message: Fix iiwa description

File: ridgeback_iiwa_description/urdf/iiwa.gazebo.xacro (robot description, xacro)
@@ -24,5 +24,4 @@
     <!-- Link0 -->
     <gazebo reference="${robot_name}_link_0">
-      <material>Gazebo/Grey</material>
       <mu1>0.2</mu1>
       <mu2>0.2</mu2>
@@ -30,5 +29,4 @@
     <!-- Link1 -->
     <gazebo reference="${robot_name}_link_1">
-      <material>Gazebo/Orange</material>
       <mu1>0.2</mu1>
       <mu2>0.2</mu2>
@@ -36,5 +34,4 @@
     <!-- Link2 -->
     <gazebo reference="${robot_name}_link_2">
-      <material>Gazebo/Orange</material>
       <mu1>0.2</mu1>
       <mu2>0.2</mu2>
@@ -42,5 +39,4 @@
     <!-- Link3 -->
     <gazebo reference="${robot_name}_link_3">
-      <material>Gazebo/Orange</material>
       <mu1>0.2</mu1>
       <mu2>0.2</mu2>
@@ -48,5 +44,4 @@
     <!-- Link4 -->
     <gazebo reference="${robot_name}_link_4">
-      <material>Gazebo/Orange</material>
       <mu1>0.2</mu1>
       <mu2>0.2</mu2>
@@ -54,5 +49,4 @@
     <!-- Link5 -->
     <gazebo reference="${robot_name}_link_5">
-      <material>Gazebo/Orange</material>
       <mu1>0.2</mu1>
       <mu2>0.2</mu2>
@@ -60,5 +54,4 @@
     <!-- Link6 -->
     <gazebo reference="${robot_name}_link_6">
-      <material>Gazebo/Orange</material>
       <mu1>0.2</mu1>
       <mu2>0.2</mu2>

File: ridgeback_iiwa_description/urdf/iiwa.transmission.xacro (robot description, xacro)
@@ -3,5 +3,4 @@
   <xacro:macro name="iiwa_transmission" params="hardware_interface">
     <transmission name="${robot_name}_tran_1">
-      <robotNamespace>/$</robotNamespace>
       <type>transmission_interface/SimpleTransmission</type>
       <joint name="${robot_name}_joint_1">
@@ -14,5 +13,4 @@
     </transmission>
     <transmission name="${robot_name}_tran_2">
-      <robotNamespace>/$</robotNamespace>
       <type>transmission_interface/SimpleTransmission</type>
       <joint name="${robot_name}_joint_2">
@@ -25,5 +23,4 @@
     </transmission>
     <transmission name="${robot_name}_tran_3">
-      <robotNamespace>/$</robotNamespace>
       <type>transmission_interface/SimpleTransmission</type>
       <joint name="${robot_name}_joint_3">
@@ -36,5 +33,4 @@
     </transmission>
     <transmission name="${robot_name}_tran_4">
-      <robotNamespace>/$</robotNamespace>
       <type>transmission_interface/SimpleTransmission</type>
       <joint name="${robot_name}_joint_4">
@@ -47,5 +43,4 @@
     </transmission>
     <transmission name="${robot_name}_tran_5">
-      <robotNamespace>/$</robotNamespace>
       <type>transmission_interface/SimpleTransmission</type>
       <joint name="${robot_name}_joint_5">
@@ -58,5 +53,4 @@
     </transmission>
     <transmission name="${robot_name}_tran_6">
-      <robotNamespace>/$</robotNamespace>
       <type>transmission_interface/SimpleTransmission</type>
       <joint name="${robot_name}_joint_6">
@@ -69,5 +63,4 @@
     </transmission>
     <transmission name="${robot_name}_tran_7">
-      <robotNamespace>/$</robotNamespace>
       <type>transmission_interface/SimpleTransmission</type>
       <joint name="${robot_name}_joint_7">

File: ridgeback_iiwa_description/urdf/iiwa7.xacro (robot description, xacro)
@@ -2,9 +2,9 @@
 <robot xmlns:xacro="http://www.ros.org/wiki/xacro">
   <!-- Import all Gazebo-customization elements, including Gazebo colors -->
-  <xacro:include filename="$(find iiwa_description)/urdf/iiwa.gazebo.xacro" />
+  <xacro:include filename="$(find ridgeback_iiwa_description)/urdf/iiwa.gazebo.xacro" />
   <!-- Import Transmissions -->
-  <xacro:include filename="$(find iiwa_description)/urdf/iiwa.transmission.xacro" />
+  <xacro:include filename="$(find ridgeback_iiwa_description)/urdf/iiwa.transmission.xacro" />
   <!-- Include Utilities -->
-  <xacro:include filename="$(find iiwa_description)/urdf/utilities.xacro" />
+  <xacro:include filename="$(find ridgeback_iiwa_description)/urdf/utilities.xacro" />
   <!-- some constants -->
   <xacro:property name="safety_controller_k_pos" value="100" />

File: ridgeback_iiwa_description/urdf/ridgeback_iiwa_robot.urdf.xacro (robot description, xacro)
@@ -4,4 +4,5 @@
   <!-- Include iiwa URDF -->
   <xacro:include filename="$(find ridgeback_iiwa_description)/urdf/iiwa7.xacro"/>
+  <!-- Include acc URDF -->
   <xacro:include filename="$(find ridgeback_iiwa_description)/urdf/hams.urdf.xacro"/>
   <xacro:arg name="hardware_interface" default="PositionJointInterface"/>
